Commit message: phc hw DONE (not working 100p tho)

File: body.urdf (robot description, URDF)
Before this commit: robot robot, 3 links, 2 joints
Links:
- removed link backLeg
- removed link frontLeg
- removed link torso
- added link BackLeg, mass 1; collision box size=1 1 1; visual box size=1 1 1
- added link FrontLeg, mass 1; collision box size=1 1 1; visual box size=1 1 1
- added link Torso, mass 1; collision box size=1 1 1; visual box size=1 1 1
Joints:
- removed joint torso_backLeg
- removed joint torso_frontLeg
- added joint Torso_BackLeg: type revolute, parent Torso, child BackLeg, origin xyz=-0.5 0 1 rpy=0 0 0, axis 0 1 0, limit lower=-3.14159 upper=3.14159 effort=0.0 velocity=0.0
- added joint Torso_FrontLeg: type revolute, parent Torso, child FrontLeg, origin xyz=0.5 0 1 rpy=0 0 0, axis 0 1 0, limit lower=-3.14159 upper=3.14159 effort=0.0 velocity=0.0
